File: hw/Mushroom.kicad_pcb (KiCad board)
At the start: 2 copper layers, 30 x 30 mm, 25 parts, among them J1 USB_C_Receptacle_PowerOnly_6P, J2 Conn_01x03, J4 Conn_01x04, U1 STM32G030F6Px, U2 LPS22HH, U3 SHT30-DIS, U4 BH1750FVI-TR, U5 SPX3819M5-L-3-3

Commit message: Finish board design
Parts:
- added J3: Conn_01x12, Mushroom_footprints:Arc_Pins_12, F.Cu at (80.0, 45.0)
- moved J2 7.42 mm to (67.0, 42.5)
- moved R6 6.80 mm to (69.4, 45.0)
Routing:
- net /TOUCH_6: track 4.75 -> 17.4 mm
- net /TOUCH_7: track 4.46 -> 15.4 mm
- net /TOUCH_4: track 5.21 -> 14.9 mm
- net /TOUCH_5: track 5.03 -> 14.4 mm
- net /TOUCH_8: track 4.36 -> 12.9 mm
- net /TOUCH_0: track 5.56 -> 13.4 mm
- net /TOUCH_2: track 3.56 -> 10.7 mm
- net /TOUCH_9: track 4.57 -> 11.5 mm
- net /TOUCH_1: track 6.22 -> 12.9 mm
- net /LED_OUT: track 6.69 -> 13.3 mm
- net /TOUCH_10: track 5.15 -> 11.6 mm
- net /TOUCH_3: track 2.85 -> 9.13 mm
- net /SWDIO: track 8.56 -> 12.9 mm
- net +5V: track 49.7 -> 48.4 mm

Commit message: Revise and finalise board design
Parts:
- added G***: LOGO, LOGO, B.Cu at (73.9, 51.9)
- added G***: LOGO, LOGO, B.Cu at (78.9, 51.7)
Routing:
- net GND: track 22.7 -> 21.3 mm, vias 17 -> 16
- added copper zone on F.Cu, net +3V3
- added copper zone on F.Cu, net +5V
- added copper zone on F.Cu, net /SDA
Other:
- board text added: "<24-Chill"
- board text added: ">"
- board text added: "Rev. 1"

Commit message: 🎉 Submit for fab (Rev. 1)
Parts:
- moved G*** 0.20 mm to (74.1, 51.9)
- moved G*** 0.20 mm to (79.1, 51.7)
Other:
- board text added: "To build resulting board: - Round tracks - Change tolerances to 0.1 mm - Add teardrops - Refill, DRC"
